File: Hardware/rSens_DIL/rSens.kicad_pcb (KiCad board)
At the start: 2 copper layers, 48.5 x 24.9 mm, 12 parts, among them J1 TO_ARDUINO, J2 RESISTIVE_SENSOR, U1 MCP602

Commit message: FIX 3D
Other:
- board outline removed
