File: Hardware/rSens_SMD/rSens.kicad_pcb (KiCad board)
At the start: 2 copper layers, 48.5 x 24.9 mm, 18 parts, among them U2 MCP6244

Commit message: Routing in progress
Parts:
- added J1: Conn_01x02, rSens:rSens_Pad_1x02, F.Cu at (127.8, 101.0)
- added J2: Conn_01x02, rSens:rSens_Pad_1x02, F.Cu at (158.8, 101.0)
- added J3: Conn_01x04, rSens:rSens_Pad_1x04, F.Cu at (140.6, 79.4)
- C1, C2, C3: footprint Capacitor_SMD:C_0603_1608Metric -> Capacitor_SMD:C_0805_2012Metric_Pad1.18x1.45mm_HandSolder
- R1, R10: footprint Resistor_SMD:R_0603_1608Metric -> Resistor_THT:R_Axial_DIN0309_L9.0mm_D3.2mm_P12.70mm_Horizontal
- R2, R3, R4, R5, R6, R7, R8, R9: footprint Resistor_SMD:R_0603_1608Metric -> Resistor_SMD:R_0805_2012Metric_Pad1.20x1.40mm_HandSolder
- moved RV2 29.0 mm to (135.3, 88.3), turned to 180 degrees
- moved R7 27.6 mm to (150.3, 106.0), turned to 180 degrees
- moved RV1 25.0 mm to (135.3, 101.0), turned to 180 degrees
- moved R3 21.7 mm to (135.3, 106.0), turned to 0 degrees
- moved R6 18.9 mm to (145.3, 106.0)
- moved RV3 18.5 mm to (151.3, 101.0), turned to 180 degrees
- moved C2 17.0 mm to (135.3, 93.0), turned to 0 degrees
- moved R4 16.7 mm to (135.3, 95.0), turned to 0 degrees
- moved R1 15.5 mm to (141.3, 96.6)
- moved R5 14.7 mm to (135.3, 97.0), turned to 180 degrees
- moved C1 14.0 mm to (151.4, 83.9)
- moved R2 11.5 mm to (140.3, 106.0)
- moved R10 11.0 mm to (145.3, 96.6), turned to 90 degrees
- moved R9 9.27 mm to (151.3, 97.0), turned to 180 degrees
- moved C3 9.23 mm to (151.3, 93.0)
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Connections:
- R10 pad 1: Net-(C3-Pad2) -> SENSOR_INPUT_B
- R10 pad 2: Net-(R10-Pad2) -> GND
- R8 pad 1: SENSOR_INPUT_B -> Net-(R8-Pad1)
- R8 pad 2: GND -> Net-(C3-Pad2)
- R9 pad 1: Net-(R9-Pad1) -> Net-(C3-Pad2)
- R9 pad 2: Net-(C3-Pad2) -> Net-(R9-Pad2)
- RV4 pad 1: Net-(R9-Pad1) -> Net-(R8-Pad1)
- U2 pad 13: Net-(R10-Pad2) -> Net-(R9-Pad2)
- U2 pad 14: Net-(R10-Pad2) -> Net-(R9-Pad2)
Routing:
- net VOLTAGE_OUTPUT_A: track 0.00 -> 16.5 mm
- net Net-(R5-Pad2): track 0.00 -> 11.9 mm
- net Net-(R3-Pad1): track 0.00 -> 9.92 mm
- net VCC: track 0.00 -> 9.78 mm
- net Net-(C2-Pad2): track 0.00 -> 9.27 mm
- net Net-(R2-Pad2): track 0.00 -> 8.68 mm
- net SENSOR_INPUT_B: track 0.00 -> 7.67 mm
- net Net-(R4-Pad1): track 0.00 -> 7.35 mm
- net Net-(R8-Pad1): track 0.00 -> 6.91 mm
- net SENSOR_INPUT_A: track 0.00 -> 5.84 mm
- net Net-(R9-Pad2): track 0.00 -> 5.64 mm
- net VOLTAGE_OUTPUT_B: track 0.00 -> 5.27 mm
- net Net-(R6-Pad2): track 0.00 -> 5.09 mm
- net Net-(C3-Pad2): track 0.00 -> 4.00 mm
- net Net-(RV1-Pad2): track 0.00 -> 3.41 mm
- added copper zone on F.Cu, net GND
Other:
- board outline removed
- net class Default: trace_width 1 -> 0.4

Commit message: Routing done
Parts:
- removed J3: Conn_01x04, rSens:rSens_Pad_1x04
- J1, J2: value Conn_01x02 -> Conn_01x04; footprint rSens:rSens_Pad_1x02 -> rSens:rSens_Pad_1x04
- moved J1 28.3 mm to (143.2, 77.3), turned to 0 degrees
- moved J2 18.7 mm to (143.2, 111.2), turned to 180 degrees
- moved C1 1.58 mm to (152.7, 84.8), turned to 0 degrees
- moved R2 0.91 mm to (140.3, 105.1)
- moved R3 0.91 mm to (135.3, 105.1)
- moved R6 0.91 mm to (145.3, 105.1)
- moved R7 0.91 mm to (150.3, 105.1)
- moved RV4 0.51 mm to (151.3, 88.8)
- moved RV2 0.51 mm to (135.3, 88.8)
Connections:
- J2 pad 1: VCC -> GND
- J2 pad 2: SENSOR_INPUT_B -> VOLTAGE_OUTPUT_B
Routing:
- net VCC: track 9.78 -> 81.6 mm, vias 0 -> 2
- net VOLTAGE_OUTPUT_B: track 5.27 -> 36.9 mm, vias 0 -> 2
- net SENSOR_INPUT_B: track 7.67 -> 26.6 mm, vias 0 -> 1
- net SENSOR_INPUT_A: track 5.84 -> 23.6 mm, vias 0 -> 1
- net Net-(C3-Pad2): track 4.00 -> 20.3 mm, vias 0 -> 2
- net VOLTAGE_OUTPUT_A: track 16.5 -> 29.2 mm, vias 0 -> 2
- net Net-(RV3-Pad2): track 0.00 -> 10.4 mm
- net Net-(R7-Pad1): track 0.00 -> 6.89 mm
- net GND: track 0.00 -> 4.85 mm, vias 0 -> 8
- net Net-(R3-Pad1): track 9.92 -> 8.36 mm
- net Net-(R6-Pad2): track 5.09 -> 4.42 mm
- net Net-(R2-Pad2): track 8.68 -> 8.04 mm
- net Net-(R4-Pad1): track 7.35 -> 6.84 mm
Other:
- board outline added: 25.4 x 33.9 mm
- board text added: "A0"
- board text added: "A1"
- board text added: "Gain"

Commit message: Added GERBER
Routing:
- net GND: track 4.85 -> 6.86 mm, vias 8 -> 10
- net VCC: track 81.6 -> 81.0 mm
Other:
- board text added: "eTextile.org"
- board text added: "rSens V1.0"
Changed lines of the file:
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@@
 (kicad_pcb (version 20171130) (host pcbnew 5.0.2+dfsg1-1)
   (general
-    (thickness 1.6)
-    (drawings 175)
-    (tracks 168)
+    (thickness 1.2)
+    (drawings 177)
+    (tracks 169)
     (zones 0)
     (modules 20)
@@
   )
   (layers
-    (0 F.Cu signal hide)
+    (0 F.Cu signal)
     (31 B.Cu power)
     (33 F.Adhes user)
     (35 F.Paste user)
+    (36 B.SilkS user)
     (37 F.SilkS user)
     (39 F.Mask user)
@@
     (solder_mask_min_width 0.25)
     (aux_axis_origin 0 0)
-    (grid_origin 134.484 108.286)
+    (grid_origin 155.884 77.277)
     (visible_elements FFFFFF7F)
     (pcbplotparams
@@
     )
   )
-  (gr_line (start 93.054009 77.877993) (end 105.584 77.877993) (layer F.Mask) (width 2))
-  (gr_line (start 105.59123 77.876) (end 105.59123 65.248884) (layer F.Mask) (width 2))
-  (gr_line (start 93.054009 70.884823) (end 105.574 70.884823) (layer F.Mask) (width 2))
-  (gr_line (start 93.054009 74.38141) (end 105.584 74.38141) (layer F.Mask) (width 2))
-  (gr_line (start 102.117616 77.866) (end 102.117616 65.248884) (layer F.Mask) (width 2))
-  (gr_line (start 98.644 77.876) (end 98.644 65.248884) (layer F.Mask) (width 2))
+  (gr_text eTextile.org (at 150.364 94.976 90) (layer B.SilkS)
+    (effects (font (size 2.5 2.5) (thickness 0.4)) (justify mirror))
+  )
+  (gr_text "rSens V1.0" (at 153.364 93.306 90) (layer B.SilkS)
+    (effects (font (size 2 2) (thickness 0.2)) (justify mirror))
+  )
+  (gr_line (start 146.962498 100.489862) (end 146.962498 87.959871) (layer B.SilkS) (width 2))
+  (gr_line (start 146.960505 87.952641) (end 134.333389 87.952641) (layer B.SilkS) (width 2))
+  (gr_line (start 139.969328 100.489862) (end 139.969328 87.969871) (layer B.SilkS) (width 2))
+  (gr_line (start 143.465915 100.489862) (end 143.465915 87.959871) (layer B.SilkS) (width 2))
+  (gr_line (start 146.950505 91.426255) (end 134.333389 91.426255) (layer B.SilkS) (width 2))
+  (gr_line (start 146.960505 94.899871) (end 134.333389 94.899871) (layer B.SilkS) (width 2))
   (gr_line (start 136.314 106.452574) (end 136.314 107.506) (layer F.Mask) (width 0.2))
   (gr_line (start 137.025077 107.4387) (end 136.974931 107.5026) (layer F.Mask) (width 0.2))
@@
   (gr_line (start 130.484 111.186) (end 155.884 111.186) (layer Edge.Cuts) (width 0.2))
   (segment (start 149.334 105.09) (end 149.334 106.764) (width 0.4) (layer F.Cu) (net 1))
-  (segment (start 150.362 106.764) (end 151.884 108.286) (width 0.9) (layer F.Cu) (net 1))
+  (segment (start 150.362 106.764) (end 151.884 108.286) (width 0.8) (layer F.Cu) (net 1))
   (segment (start 149.334 106.764) (end 150.362 106.764) (width 0.4) (layer F.Cu) (net 1))
   (via (at 136.802 83.754) (size 0.8) (drill 0.4) (layers F.Cu B.Cu) (net 1))
-  (via (at 146.962 90.485) (size 0.8) (drill 0.4) (layers F.Cu B.Cu) (net 1))
-  (via (at 143.66 93.787) (size 0.8) (drill 0.4) (layers F.Cu B.Cu) (net 1))
+  (via (at 146.2574 91.2851) (size 0.8) (drill 0.4) (layers F.Cu B.Cu) (net 1))
   (via (at 139.850001 90.865999) (size 0.8) (drill 0.4) (layers F.Cu B.Cu) (net 1))
   (via (at 137.31 109.535) (size 0.8) (drill 0.4) (layers F.Cu B.Cu) (net 1))
@@
   (via (at 131.648 104.984) (size 0.8) (drill 0.4) (layers F.Cu B.Cu) (net 1))
   (via (at 137.31 91.374) (size 0.8) (drill 0.4) (layers F.Cu B.Cu) (net 1))
+  (via (at 153.874 105.09) (size 0.8) (drill 0.4) (layers F.Cu B.Cu) (net 1))
+  (via (at 132.4017 95.946) (size 0.8) (drill 0.4) (layers F.Cu B.Cu) (net 1))
+  (via (at 146.2447 94.2188) (size 0.8) (drill 0.4) (layers F.Cu B.Cu) (net 1))
+  (segment (start 151.884 108.286) (end 153.302 106.868) (width 0.8) (layer F.Cu) (net 1))
   (segment (start 137.984 101.646) (end 137.334 100.996) (width 0.4) (layer F.Cu) (net 2))
   (segment (start 140.4715 101.646) (end 137.984 101.646) (width 0.4) (layer F.Cu) (net 2))
@@
   (segment (start 134.484 97.629) (end 134.484 105.09) (width 0.4) (layer B.Cu) (net 4))
   (segment (start 134.484 105.09) (end 134.484 107.305262) (width 0.4) (layer B.Cu) (net 4))
-  (segment (start 134.484 105.09) (end 139.088 105.09) (width 0.4) (layer B.Cu) (net 4))
-  (segment (start 139.958001 104.219999) (end 140.358 103.82) (width 0.4) (layer B.Cu) (net 4))
-  (segment (start 139.088 105.09) (end 139.958001 104.219999) (width 0.4) (layer B.Cu) (net 4))
   (via (at 140.358 103.82) (size 0.8) (drill 0.4) (layers F.Cu B.Cu) (net 4))
   (segment (start 141.334 105.09) (end 141.334 104.256) (width 0.4) (layer F.Cu) (net 4))
@@
   (segment (start 140.4715 100.996) (end 141.602 100.996) (width 0.4) (layer F.Cu) (net 4))
   (segment (start 141.602 100.996) (end 142.009 101.403) (width 0.4) (layer F.Cu) (net 4))
+  (segment (start 134.548 103.82) (end 140.358 103.82) (width 0.4) (layer B.Cu) (net 4))
   (segment (start 139.334 104.384) (end 139.334 104.996) (width 0.4) (layer F.Cu) (net 5))
   (segment (start 138.77 103.82) (end 139.334 104.384) (width 0.4) (layer F.Cu) (net 5))
